File: KeyCade Cartridge.brd (EAGLE design)
At the start: 10.8 x 9.2 mm, 2 parts, among them U1 EEPROM-I2CSMD

Commit message: Aestheric updates
Initial Checkin
Parts:
- added FRAME1: FRAME-LETTER, StuffLabs:CREATIVE_COMMONS
Changed lines of the file:
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@@
 <layer number="230" name="230bmp" color="7" fill="1" visible="no" active="yes"/>
 <layer number="231" name="231bmp" color="7" fill="1" visible="no" active="yes"/>
+<layer number="232" name="Eagle3D_PG2" color="14" fill="2" visible="yes" active="yes"/>
+<layer number="233" name="Eagle3D_PG3" color="14" fill="4" visible="yes" active="yes"/>
 <layer number="248" name="Housing" color="7" fill="1" visible="yes" active="yes"/>
 <layer number="249" name="Edge" color="7" fill="1" visible="yes" active="yes"/>
@@
 </element>
 <element name="U1" library="SparkFun-DigitalIC" package="SO08" value="EEPROM-I2CSMD" x="5.3975" y="6.0325" smashed="yes" rot="R270"/>
+<element name="FRAME1" library="StuffLabs" package="CREATIVE_COMMONS" value="FRAME-LETTER" x="13.97" y="-16.51"/>
 </elements>
 <signals>
