File: KeyCade Cartridge.sch (EAGLE design)
At the start: 2 parts, among them U1 EEPROM-I2CSMD

Commit message: Aestheric updates
Initial Checkin
Parts:
- added FRAME1: FRAME-LETTER, StuffLabs:FRAME-LETTER
Changed lines of the file:
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@@
 <layer number="230" name="230bmp" color="7" fill="1" visible="yes" active="yes"/>
 <layer number="231" name="231bmp" color="7" fill="1" visible="yes" active="yes"/>
+<layer number="232" name="Eagle3D_PG2" color="14" fill="2" visible="yes" active="yes"/>
+<layer number="233" name="Eagle3D_PG3" color="14" fill="4" visible="yes" active="yes"/>
 <layer number="248" name="Housing" color="7" fill="1" visible="yes" active="yes"/>
 <layer number="249" name="Edge" color="7" fill="1" visible="yes" active="yes"/>
@@
 <part name="P+1" library="supply1" deviceset="VCC" device=""/>
 <part name="P+2" library="supply1" deviceset="VCC" device=""/>
+<part name="FRAME1" library="StuffLabs" deviceset="FRAME-LETTER" device=""/>
 </parts>
 <sheets>
@@
 <instance part="P+1" gate="VCC" x="114.3" y="66.04"/>
 <instance part="P+2" gate="VCC" x="76.2" y="33.02"/>
+<instance part="FRAME1" gate="G$1" x="-33.02" y="-45.72"/>
+<instance part="FRAME1" gate="V" x="114.3" y="-45.72"/>
 </instances>
 <busses>
