File: KeyCade.brd (EAGLE design)
At the start: 27 x 41 mm, 22 parts, among them SW2 SPST_TACT-EVQQ2, SW3 SPST_TACT-EVQQ2, Y1 CRYSTALSMD3215

Commit message: Aestheric updates
Initial Checkin
Parts:
- added FRAME1: FRAME-LETTER, StuffLabs:CREATIVE_COMMONS
Changed lines of the file:
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@@
 <attribute name="VALUE" x="7.27075" y="38.1635" size="0.0254" layer="28" rot="MR0"/>
 </element>
+<element name="FRAME1" library="StuffLabs" package="CREATIVE_COMMONS" value="FRAME-LETTER" x="13.335" y="-10.795"/>
 </elements>
 <signals>
