File: KeyCade.sch (EAGLE design)
At the start: 22 parts, among them SW2 SPST_TACT-EVQQ2, SW3 SPST_TACT-EVQQ2, Y1 CRYSTALSMD3215

Commit message: Aestheric updates
Initial Checkin
Parts:
- added FRAME1: FRAME-LETTER, StuffLabs:FRAME-LETTER
Other:
- moved on the sheet: BAT1, C1, C2, C3, C4, C5, CART, GND, LCD, R1, R4, RX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
